Commit message: Rename package folder/paths from ASm13.SLDASM to Robot67.SLDASM

File: Robot67.SLDASM/urdf/Robot67.SLDASM.urdf (robot description, URDF)
Before this commit: robot ASm13.SLDASM, 4 links, 3 joints
Links:
- link Link1: geometry collision mesh filename=package://Robot67.SLDASM/meshes/Link1.STL; visual mesh filename=package://Robot67.SLDASM/meshes/Link1.STL
- link Link2: geometry collision mesh filename=package://Robot67.SLDASM/meshes/Link2.STL; visual mesh filename=package://Robot67.SLDASM/meshes/Link2.STL
- link Link3: geometry collision mesh filename=package://Robot67.SLDASM/meshes/Link3.STL; visual mesh filename=package://Robot67.SLDASM/meshes/Link3.STL
- link base_link: geometry collision mesh filename=package://Robot67.SLDASM/meshes/base_link.STL; visual mesh filename=package://Robot67.SLDASM/meshes/base_link.STL
